Commit message: nav2 moving with mujoco pose
Co-Authored-By: Claude Opus 4.6 <noreply@anthropic.com>

File: ros2_ws/src/tidybot_description/urdf/tidybot_wx250s.urdf.xacro (robot description, xacro)
@@ -34,7 +34,15 @@
   <!-- Odom frame for mobile base -->
   <link name="odom"/>
-  <joint name="odom_to_base" type="floating">
+  <link name="base_footprint"/>
+  <joint name="odom_to_base_footprint" type="floating">
     <parent link="odom"/>
+    <child link="base_footprint"/>
+  </joint>
+  <!-- base_footprint follows ROS convention (+X = forward).
+       base_link is rotated 90° because the URDF mesh faces -Y. -->
+  <joint name="base_footprint_to_base_link" type="fixed">
+    <parent link="base_footprint"/>
     <child link="base_link"/>
+    <origin xyz="0 0 0" rpy="0 0 1.5708"/>
   </joint>
   <!-- ==================== CAMERA MOUNT ==================== -->
