Commit message: Fixed gripper sim issues, added midding forearm_roll

File: ros2_ws/src/tidybot_description/urdf/tidybot_wx250s.urdf.xacro (robot description, xacro)
@@ -330,5 +330,5 @@
       <origin xyz="0 0.015 0" rpy="0 0 0"/>
       <axis xyz="0 1 0"/>
-      <limit lower="0" upper="0.037" effort="5" velocity="1"/>
+      <limit lower="-0.014" upper="0.022" effort="5" velocity="1"/>
       <dynamics damping="0.1"/>
     </joint>
@@ -353,5 +353,5 @@
       <origin xyz="0 -0.015 0" rpy="0 0 0"/>
       <axis xyz="0 -1 0"/>
-      <limit lower="0" upper="0.037" effort="5" velocity="1"/>
+      <limit lower="-0.014" upper="0.022" effort="5" velocity="1"/>
       <dynamics damping="0.1"/>
     </joint>

Commit message: Added Lidar Model Updates

File: ros2_ws/src/tidybot_description/urdf/tidybot_wx250s.urdf.xacro (robot description, xacro)
@@ -57,4 +57,81 @@
     <origin xyz="0 -0.1125 0.279" rpy="0 0 -1.5708"/>
   </joint>
+  <!-- ==================== LIDAR STACK (EXTRUSION + MOUNT + LIDAR) ==================== -->
+  <link name="lidar_extrusion">
+    <visual>
+      <geometry>
+        <!-- This STL is already in meters -->
+        <mesh filename="${mesh_path}/base/2020_Aluminum_Extrusion_400mm.stl" scale="1 1 1"/>
+      </geometry>
+      <material name="silver"/>
+    </visual>
+    <inertial>
+      <origin xyz="0 0 0"/>
+      <mass value="0.6"/>
+      <inertia ixx="0.001" ixy="0" ixz="0" iyy="0.001" iyz="0" izz="0.001"/>
+    </inertial>
+  </link>
+  <joint name="base_to_lidar_extrusion" type="fixed">
+    <parent link="base_link"/>
+    <child link="lidar_extrusion"/>
+    <!-- Requested placement: x=0, y=190mm in base_link frame -->
+    <origin xyz="0.0 0.196 0.5471" rpy="0 0 0"/>
+  </joint>
+  <link name="lidar_mount">
+    <visual>
+      <!-- Keep mesh orientation unchanged while mount frame is reoriented -->
+      <origin xyz="0 0 0" rpy="-1.5708 0 0"/>
+      <geometry>
+        <!-- This STL is already in meters -->
+        <mesh filename="${mesh_path}/base/Lidar_Mount.stl" scale="1 1 1"/>
+      </geometry>
+      <material name="dark_grey"/>
+    </visual>
+    <inertial>
+      <origin xyz="0 0 0"/>
+      <mass value="0.1"/>
+      <inertia ixx="0.0001" ixy="0" ixz="0" iyy="0.0001" iyz="0" izz="0.0001"/>
+    </inertial>
+  </link>
+  <joint name="lidar_extrusion_to_mount" type="fixed">
+    <parent link="lidar_extrusion"/>
+    <child link="lidar_mount"/>
+    <!-- Reorient mount frame so z_new aligns with +z_base (old z -> old -y) -->
+    <origin xyz="0 0 0.229" rpy="0 0 0"/>
+  </joint>
+  <link name="lidar_link">
+    <visual>
+      <origin xyz="0 0 0" rpy="0 0 0"/>
+      <geometry>
+        <mesh filename="${mesh_path}/base/locobot_lidar.stl" scale="0.001 0.001 0.001"/>
+      </geometry>
+      <material name="dark_grey"/>
+    </visual>
+    <collision>
+      <origin xyz="0 0 -0.0091" rpy="0 0 0"/>
+      <geometry>
+        <cylinder radius="0.03785" length="0.0408"/>
+      </geometry>
+    </collision>
+    <inertial>
+      <origin xyz="0.0007379970 0 -0.0103809000" rpy="0 0 0"/>
+      <mass value="0.196"/>
+      <inertia ixx="0.0000907500" ixy="0.0000000001" ixz="-0.0000014234"
+               iyy="0.0000877600" iyz="0" izz="0.0001268000"/>
+    </inertial>
+  </link>
+  <joint name="lidar_mount_to_lidar" type="fixed">
+    <parent link="lidar_mount"/>
+    <child link="lidar_link"/>
+    <!-- z_lidar aligns with +z_base_link; x_lidar points toward +y_base_link -->
+    <origin xyz="0 0 0.029" rpy="0 0 1.5708"/>
+  </joint>
+  <!-- Match RPLIDAR frame_id:=laser from real.launch.py -->
+  <link name="laser"/>
+  <joint name="lidar_to_laser" type="fixed">
+    <parent link="lidar_link"/>
+    <child link="laser"/>
+    <origin xyz="0 0 0" rpy="0 0 0"/>
+  </joint>
   <!-- ==================== PAN-TILT CAMERA SYSTEM ==================== -->
   <link name="pan_link">
@@ -152,5 +229,5 @@
       <parent link="base_link"/>
       <child link="${prefix}_arm_base_link"/>
-      <origin xyz="${x_offset} ${y_offset} 0.3847" rpy="0 0 ${yaw}"/>
+      <origin xyz="${x_offset} ${y_offset} 0.3817" rpy="0 0 ${yaw}"/>
     </joint>
     <link name="${prefix}_shoulder_link">

Commit message: Adjusted tf for top camera so that it can be used

File: ros2_ws/src/tidybot_description/urdf/tidybot_wx250s.urdf.xacro (robot description, xacro)
@@ -57,5 +57,5 @@
     <origin xyz="0 -0.1125 0.279" rpy="0 0 -1.5708"/>
   </joint>
-  <!-- ==================== TOP CAMERA STACK (EXTRUSION + MOUNT + CAMERA) ==================== -->
+  <!-- ==================== TOP SENSOR STACK (SHARED EXTRUSION + LIDAR + TOP CAMERA) ==================== -->
   <link name="top_camera_extrusion">
     <visual>
@@ -75,9 +75,82 @@
     <parent link="base_link"/>
     <child link="top_camera_extrusion"/>
-    <!-- Initial placement reuses prior lidar stack pose -->
+    <!-- Shared top-sensor extrusion placement -->
     <origin xyz="0.0 0.196 0.5471" rpy="0 0 0"/>
   </joint>
+  <link name="lidar_mount">
+    <visual>
+      <origin xyz="0 0 0" rpy="-1.5708 0 0"/>
+      <geometry>
+        <mesh filename="${mesh_path}/base/Lidar_Mount.stl" scale="1 1 1"/>
+      </geometry>
+      <material name="dark_grey"/>
+    </visual>
+    <inertial>
+      <origin xyz="0 0 0"/>
+      <mass value="0.1"/>
+      <inertia ixx="0.0001" ixy="0" ixz="0" iyy="0.0001" iyz="0" izz="0.0001"/>
+    </inertial>
+  </link>
+  <joint name="top_camera_extrusion_to_lidar_mount" type="fixed">
+    <parent link="top_camera_extrusion"/>
+    <child link="lidar_mount"/>
+    <origin xyz="0 0 0.237" rpy="0 0 0"/>
+  </joint>
+  <link name="lidar_link">
+    <visual>
+      <origin xyz="0 0 0" rpy="0 0 0"/>
+      <geometry>
+        <mesh filename="${mesh_path}/base/locobot_lidar.stl" scale="0.001 0.001 0.001"/>
+      </geometry>
+      <material name="dark_grey"/>
+    </visual>
+    <collision>
+      <origin xyz="0 0 -0.0091" rpy="0 0 0"/>
+      <geometry>
+        <cylinder radius="0.03785" length="0.0408"/>
+      </geometry>
+    </collision>
+    <inertial>
+      <origin xyz="0.0007379970 0 -0.0103809000" rpy="0 0 0"/>
+      <mass value="0.196"/>
+      <inertia ixx="0.0000907500" ixy="0.0000000001" ixz="-0.0000014234"
+               iyy="0.0000877600" iyz="0" izz="0.0001268000"/>
+    </inertial>
+  </link>
+  <joint name="lidar_mount_to_lidar" type="fixed">
+    <parent link="lidar_mount"/>
+    <child link="lidar_link"/>
+    <origin xyz="0 0 0.029" rpy="0 0 1.5708"/>
+  </joint>
+  <link name="laser"/>
+  <joint name="lidar_to_laser" type="fixed">
+    <parent link="lidar_link"/>
+    <child link="laser"/>
+    <origin xyz="0 0 0" rpy="0 0 0"/>
+  </joint>
+  <link name="top_camera_mount">
+    <visual>
+      <!-- Rotate the STL in its own frame without changing the mount link frame. -->
+      <origin xyz="0 0 0" rpy="1.5708 0 0"/>
+      <geometry>
+        <mesh filename="${mesh_path}/base/top_camera_mount_20deg.stl" scale="0.001 0.001 0.001"/>
+      </geometry>
+      <material name="dark_grey"/>
+    </visual>
+    <inertial>
+      <origin xyz="0 0 0"/>
+      <mass value="0.1"/>
+      <inertia ixx="0.0001" ixy="0" ixz="0" iyy="0.0001" iyz="0" izz="0.0001"/>
+    </inertial>
+  </link>
+  <joint name="top_camera_extrusion_to_mount" type="fixed">
+    <parent link="top_camera_extrusion"/>
+    <child link="top_camera_mount"/>
+    <origin xyz="0 -0.011 0.150454" rpy="0 0 -1.5708"/>
+  </joint>
   <link name="top_camera_link">
     <visual>
+      <!-- Place top_camera_link at the center of the camera back plate. -->
+      <origin xyz="0.02078 0.0175 0" rpy="0 0 0"/>
       <geometry>
         <mesh filename="${mesh_path}/locobot_pantilt/locobot_camera.stl" scale="0.001 0.001 0.001"/>
@@ -86,17 +159,13 @@
     </visual>
     <inertial>
-      <origin xyz="-0.008972 -0.015818 0.000003"/>
+      <origin xyz="0.011808 0.001682 0.000003"/>
       <mass value="0.072"/>
       <inertia ixx="0.0000465400" ixy="0" ixz="0" iyy="0.0000069128" iyz="0" izz="0.0000468600"/>
     </inertial>
   </link>
-  <joint name="top_camera_extrusion_to_camera" type="fixed">
-    <parent link="top_camera_extrusion"/>
+  <joint name="top_camera_mount_to_camera" type="fixed">
+    <parent link="top_camera_mount"/>
     <child link="top_camera_link"/>
-    <!-- Mount target:
-         - 40 mm forward
-         - 65 mm above top surface of the 400 mm extrusion
-         - 20 deg downward tilt -->
-    <origin xyz="0 -0.04 0.135" rpy="0 0.3491 -1.5708"/>
+    <origin xyz="0.0097 0 0.013155 " rpy="0 0.3491 0"/>
   </joint>
   <!-- ==================== PAN-TILT CAMERA SYSTEM ==================== -->

Commit message: Updated urdf to have valid top_camera lens frames

File: ros2_ws/src/tidybot_description/urdf/tidybot_wx250s.urdf.xacro (robot description, xacro)
@@ -151,6 +151,6 @@
   <link name="top_camera_link">
     <visual>
-      <!-- Place top_camera_link at the center of the camera back plate. -->
-      <origin xyz="0.02078 0.0175 0" rpy="0 0 0"/>
+      <!-- Keep top_camera_link at the camera mesh center (same convention as camera_link). -->
+      <origin xyz="0 0 0" rpy="0 0 0"/>
       <geometry>
         <mesh filename="${mesh_path}/locobot_pantilt/locobot_camera.stl" scale="0.001 0.001 0.001"/>
@@ -167,5 +167,6 @@
     <parent link="top_camera_mount"/>
     <child link="top_camera_link"/>
-    <origin xyz="0.0097 0 0.013155 " rpy="0 0.3491 0"/>
+    <!-- Adjusted so camera mesh pose remains consistent after moving link origin to mesh center. -->
+    <origin xyz="0.029227 0.0175 0.006047" rpy="0 0.3491 0"/>
   </joint>
   <!-- ==================== PAN-TILT CAMERA SYSTEM ==================== -->

Commit message: Update tidybot_wx250s.urdf.xacro

File: ros2_ws/src/tidybot_description/urdf/tidybot_wx250s.urdf.xacro (robot description, xacro)
@@ -55,5 +55,5 @@
     <parent link="base_link"/>
     <child link="camera_mount"/>
-    <origin xyz="0 -0.1125 0.279" rpy="0 0 -1.5708"/>
+    <origin xyz="0 -0.1125 0.279" rpy="0 0 0"/>
   </joint>
   <!-- ==================== TOP SENSOR STACK (SHARED EXTRUSION + LIDAR + TOP CAMERA) ==================== -->
