Commit message: Integrate 2D LiDAR with Nav2 + SLAM alongside depth camera
- Add base_footprint frame to lidar URDF for Nav2 compatibility
- Support three scan_source modes: depth, lidar, both (default: both)
- Add dual observation sources (scan + scan_depth) in costmaps
- Increase SLAM max_laser_range to 8m for RPLidar A2

Co-Authored-By: Claude Opus 4.6 <noreply@anthropic.com>

File: ros2_ws/src/tidybot_description/urdf/tidybot_wx250s_lidar.urdf.xacro (robot description, xacro)
@@ -32,9 +32,15 @@
     </inertial>
   </link>
-  <!-- Odom frame for mobile base -->
+  <!-- Odom frame for mobile base (with base_footprint for Nav2) -->
   <link name="odom"/>
-  <joint name="odom_to_base" type="floating">
+  <link name="base_footprint"/>
+  <joint name="odom_to_base_footprint" type="floating">
     <parent link="odom"/>
+    <child link="base_footprint"/>
+  </joint>
+  <joint name="base_footprint_to_base_link" type="fixed">
+    <parent link="base_footprint"/>
     <child link="base_link"/>
+    <origin xyz="0 0 0" rpy="0 0 1.5708"/>
   </joint>
   <!-- ==================== CAMERA MOUNT ==================== -->
